File: extras/schematics/lora_digirepeater_micro.kicad_pcb (KiCad board)
At the start: 2 copper layers, 58.9 x 19.3 mm, 9 parts, among them J1 Conn_01x02_Male, J2 Conn_Coaxial, U1 ProMicro, U2 Ai-Thinker-Ra-01

Commit message: Added missing files
Other:
- net class Default removed
